File: PCB/ATTiny1616-S.kicad_pcb (KiCad board)
At the start: 2 copper layers, 21.7 x 29.8 mm, 15 parts, among them J1 USB_C_Receptacle_USB2.0_16P, J10 Conn_01x08_Pin, U1 XC6206PxxxMR, U2 ATtiny1616-S, U3 CH340X

Commit message: Add files via upload
Parts:
- R1, R2, R3, R4: footprint Capacitor_SMD:C_0201_0603Metric -> Resistor_SMD:R_0201_0603Metric
Changed lines of the file:
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@@
 		(property ki_fp_filters "Connector*:*_1x??_*")
 		(sheetname "/")
-		(sheetfile "resolution_w7.kicad_sch")
+		(sheetfile "ATTiny1616-S.kicad_sch")
 		(units
 			(unit
@@
 		(property ki_fp_filters "USB*C*Receptacle*")
 		(sheetname "/")
-		(sheetfile "resolution_w7.kicad_sch")
+		(sheetfile "ATTiny1616-S.kicad_sch")
 		(units
 			(unit
@@
 		(property ki_fp_filters "C_*")
 		(sheetname "/")
-		(sheetfile "resolution_w7.kicad_sch")
+		(sheetfile "ATTiny1616-S.kicad_sch")
 		(units
 			(unit
@@
 		(property ki_fp_filters "C_*")
 		(sheetname "/")
-		(sheetfile "resolution_w7.kicad_sch")
+		(sheetfile "ATTiny1616-S.kicad_sch")
 		(units
 			(unit
@@
 		(property ki_fp_filters "C_*")
 		(sheetname "/")
-		(sheetfile "resolution_w7.kicad_sch")
+		(sheetfile "ATTiny1616-S.kicad_sch")
 		(units
 			(unit
@@
 		(property ki_fp_filters "LED* LED_SMD:* LED_THT:*")
 		(sheetname "/")
-		(sheetfile "resolution_w7.kicad_sch")
+		(sheetfile "ATTiny1616-S.kicad_sch")
 		(units
 			(unit
@@
 		(property ki_fp_filters "C_*")
 		(sheetname "/")
-		(sheetfile "resolution_w7.kicad_sch")
+		(sheetfile "ATTiny1616-S.kicad_sch")
 		(units
 			(unit
@@
 		)
 	)
-	(footprint "Capacitor_SMD:C_0201_0603Metric"
+	(footprint "Resistor_SMD:R_0201_0603Metric"
 		(layer "B.Cu")
 		(at 166.98 72.825 -90)
-		(descr "Capacitor SMD 0201 (0603 Metric), square (rectangular) end terminal, IPC-7351 nominal, (Body size source: https://www.vishay.com/docs/20052/crcw0201e3.pdf)")
-		(tags "capacitor")
+		(descr "Resistor SMD 0201 (0603 Metric), square (rectangular) end terminal, IPC-7351 nominal, (Body size source: https://www.vishay.com/docs/20052/crcw0201e3.pdf)")
+		(tags "resistor")
 		(property "Reference" "R1"
-			(at -0.11 -0.65 90)
+			(at 0 1.05 90)
 			(layer "B.SilkS")
 			(effects
 				(font
-					(size 0.3 0.3)
-					(thickness 0.075)
+					(size 1 1)
+					(thickness 0.15)
 				)
 				(justify mirror)
@@
 			(at 0 -1.05 90)
 			(layer "B.Fab")
-			(hide yes)
 			(effects
 				(font
@@
 		(property ki_fp_filters "R_*")
 		(sheetname "/")
-		(sheetfile "resolution_w7.kicad_sch")
+		(sheetfile "ATTiny1616-S.kicad_sch")
 		(units
 			(unit
@@
 		)
 		(fp_text user "${REFERENCE}"
-			(at -0.125 -0.63 90)
+			(at 0 0.68 90)
 			(layer "B.Fab")
 			(effects
@@
 		)
 		(embedded_fonts no)
-		(model "${KICAD10_3DMODEL_DIR}/Capacitor_SMD.3dshapes/C_0201_0603Metric.step"
+		(model "${KICAD10_3DMODEL_DIR}/Resistor_SMD.3dshapes/R_0201_0603Metric.step"
 			(offset
 				(xyz 0 0 0)
@@
 		(property ki_fp_filters "SOIC*7.5x12.8mm*P1.27mm*")
 		(sheetname "/")
-		(sheetfile "resolution_w7.kicad_sch")
+		(sheetfile "ATTiny1616-S.kicad_sch")
 		(units
 			(unit
@@
 		)
 	)
-	(footprint "Capacitor_SMD:C_0201_0603Metric"
+	(footprint "Resistor_SMD:R_0201_0603Metric"
 		(layer "B.Cu")
 		(at 166.94 76.88 90)
-		(descr "Capacitor SMD 0201 (0603 Metric), square (rectangular) end terminal, IPC-7351 nominal, (Body size source: https://www.vishay.com/docs/20052/crcw0201e3.pdf)")
-		(tags "capacitor")
+		(descr "Resistor SMD 0201 (0603 Metric), square (rectangular) end terminal, IPC-7351 nominal, (Body size source: https://www.vishay.com/docs/20052/crcw0201e3.pdf)")
+		(tags "resistor")
 		(property "Reference" "R3"
-			(at 0.02 0.79 270)
+			(at 0 1.05 270)
 			(layer "B.SilkS")
 			(effects
 				(font
-					(size 0.3 0.3)
-					(thickness 0.075)
+					(size 1 1)
+					(thickness 0.15)
 				)
 				(justify mirror)
@@
 		(property ki_fp_filters "R_*")
 		(sheetname "/")
-		(sheetfile "resolution_w7.kicad_sch")
+		(sheetfile "ATTiny1616-S.kicad_sch")
 		(units
 			(unit
@@
 		)
 		(embedded_fonts no)
-		(model "${KICAD10_3DMODEL_DIR}/Capacitor_SMD.3dshapes/C_0201_0603Metric.step"
+		(model "${KICAD10_3DMODEL_DIR}/Resistor_SMD.3dshapes/R_0201_0603Metric.step"
 			(offset
 				(xyz 0 0 0)
@@
 		)
 	)
-	(footprint "Capacitor_SMD:C_0201_0603Metric"
+	(footprint "Resistor_SMD:R_0201_0603Metric"
 		(layer "B.Cu")
 		(at 168.64 55.6 180)
-		(descr "Capacitor SMD 0201 (0603 Metric), square (rectangular) end terminal, IPC-7351 nominal, (Body size source: https://www.vishay.com/docs/20052/crcw0201e3.pdf)")
-		(tags "capacitor")
+		(descr "Resistor SMD 0201 (0603 Metric), square (rectangular) end terminal, IPC-7351 nominal, (Body size source: https://www.vishay.com/docs/20052/crcw0201e3.pdf)")
+		(tags "resistor")
 		(property "Reference" "R4"
-			(at 0.005 0.71 0)
+			(at 0 1.05 0)
 			(layer "B.SilkS")
 			(effects
 				(font
-					(size 0.3 0.3)
-					(thickness 0.075)
+					(size 1 1)
+					(thickness 0.15)
 				)
 				(justify mirror)
@@
 			(at 0 -1.05 0)
 			(layer "B.Fab")
-			(hide yes)
 			(effects
 				(font
@@
 		(property ki_fp_filters "R_*")
 		(sheetname "/")
-		(sheetfile "resolution_w7.kicad_sch")
+		(sheetfile "ATTiny1616-S.kicad_sch")
 		(units
 			(unit
@@
 		)
 		(embedded_fonts no)
-		(model "${KICAD10_3DMODEL_DIR}/Capacitor_SMD.3dshapes/C_0201_0603Metric.step"
+		(model "${KICAD10_3DMODEL_DIR}/Resistor_SMD.3dshapes/R_0201_0603Metric.step"
 			(offset
 				(xyz 0 0 0)
@@
 		)
 	)
-	(footprint "Capacitor_SMD:C_0201_0603Metric"
+	(footprint "Resistor_SMD:R_0201_0603Metric"
 		(layer "B.Cu")
 		(at 160.76 70.86 180)
-		(descr "Capacitor SMD 0201 (0603 Metric), square (rectangular) end terminal, IPC-7351 nominal, (Body size source: https://www.vishay.com/docs/20052/crcw0201e3.pdf)")
-		(tags "capacitor")
+		(descr "Resistor SMD 0201 (0603 Metric), square (rectangular) end terminal, IPC-7351 nominal, (Body size source: https://www.vishay.com/docs/20052/crcw0201e3.pdf)")
+		(tags "resistor")
 		(property "Reference" "R2"
-			(at 1.12 -0.06 0)
+			(at 0 1.05 0)
 			(layer "B.SilkS")
 			(effects
 				(font
-					(size 0.3 0.3)
-					(thickness 0.075)
+					(size 1 1)
+					(thickness 0.15)
 				)
 				(justify mirror)
@@
 			(at 0 -1.05 0)
 			(layer "B.Fab")
-			(hide yes)
 			(effects
 				(font
@@
 		(property ki_fp_filters "R_*")
 		(sheetname "/")
-		(sheetfile "resolution_w7.kicad_sch")
+		(sheetfile "ATTiny1616-S.kicad_sch")
 		(units
 			(unit
@@
 			(layer "B.Fab")
 		)
+		(fp_text user "${REFERENCE}"
+			(at 0 0.68 0)
+			(layer "B.Fab")
+			(effects
+				(font
+					(size 0.25 0.25)
+					(thickness 0.04)
+				)
+				(justify mirror)
+			)
+		)
 		(pad "" smd roundrect
 			(at -0.345 0 180)
@@
 		)
 		(embedded_fonts no)
-		(model "${KICAD10_3DMODEL_DIR}/Capacitor_SMD.3dshapes/C_0201_0603Metric.step"
+		(model "${KICAD10_3DMODEL_DIR}/Resistor_SMD.3dshapes/R_0201_0603Metric.step"
 			(offset
 				(xyz 0 0 0)
@@
 		(property ki_fp_filters "SOT?23?3*")
 		(sheetname "/")
-		(sheetfile "resolution_w7.kicad_sch")
+		(sheetfile "ATTiny1616-S.kicad_sch")
 		(units
 			(unit
@@
 		(property ki_fp_filters "C_*")
 		(sheetname "/")
-		(sheetfile "resolution_w7.kicad_sch")
+		(sheetfile "ATTiny1616-S.kicad_sch")
 		(units
 			(unit
@@
 		(property ki_fp_filters "MSOP*3x3mm*P0.5mm*")
 		(sheetname "/")
-		(sheetfile "resolution_w7.kicad_sch")
+		(sheetfile "ATTiny1616-S.kicad_sch")
 		(units
 			(unit
