File: PCB/ATTiny1616-S.kicad_sch (KiCad schematic)
At the start: 15 parts, among them J1 USB_C_Receptacle_USB2.0_16P, J10 Conn_01x08_Pin, U1 XC6206PxxxMR, U2 ATtiny1616-S, U3 CH340X

Commit message: Add files via upload
Parts:
- R1, R2, R3, R4: footprint Capacitor_SMD:C_0201_0603Metric -> Resistor_SMD:R_0201_0603Metric
Changed lines of the file:
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@@
 		)
 		(instances
-			(project "resolution_w7"
+			(project "ATTiny1616-S"
 				(path "/ee73a050-21e3-4389-9e79-fb5dbee0e802"
 					(reference "C1")
@@
 		)
 		(instances
-			(project "resolution_w7"
+			(project "ATTiny1616-S"
 				(path "/ee73a050-21e3-4389-9e79-fb5dbee0e802"
 					(reference "#PWR01")
@@
 			)
 		)
-		(property "Footprint" "Capacitor_SMD:C_0201_0603Metric"
+		(property "Footprint" "Resistor_SMD:R_0201_0603Metric"
 			(at 92.71 71.882 90)
 			(hide yes)
@@
 		)
 		(instances
-			(project "resolution_w7"
+			(project "ATTiny1616-S"
 				(path "/ee73a050-21e3-4389-9e79-fb5dbee0e802"
 					(reference "R4")
@@
 		)
 		(instances
-			(project "resolution_w7"
+			(project "ATTiny1616-S"
 				(path "/ee73a050-21e3-4389-9e79-fb5dbee0e802"
 					(reference "C3")
@@
 		)
 		(instances
-			(project "resolution_w7"
+			(project "ATTiny1616-S"
 				(path "/ee73a050-21e3-4389-9e79-fb5dbee0e802"
 					(reference "J10")
@@
 		)
 		(instances
-			(project "resolution_w7"
+			(project "ATTiny1616-S"
 				(path "/ee73a050-21e3-4389-9e79-fb5dbee0e802"
 					(reference "#PWR09")
@@
 			)
 		)
-		(property "Footprint" "Capacitor_SMD:C_0201_0603Metric"
+		(property "Footprint" "Resistor_SMD:R_0201_0603Metric"
 			(at 59.69 42.418 90)
 			(hide yes)
@@
 		)
 		(instances
-			(project "resolution_w7"
+			(project "ATTiny1616-S"
 				(path "/ee73a050-21e3-4389-9e79-fb5dbee0e802"
 					(reference "R2")
@@
 		)
 		(instances
-			(project "resolution_w7"
+			(project "ATTiny1616-S"
 				(path "/ee73a050-21e3-4389-9e79-fb5dbee0e802"
 					(reference "C5")
@@
 		)
 		(instances
-			(project "resolution_w7"
+			(project "ATTiny1616-S"
 				(path "/ee73a050-21e3-4389-9e79-fb5dbee0e802"
 					(reference "U1")
@@
 		)
 		(instances
-			(project "resolution_w7"
+			(project "ATTiny1616-S"
 				(path "/ee73a050-21e3-4389-9e79-fb5dbee0e802"
 					(reference "J1")
@@
 			)
 		)
-		(property "Footprint" "Capacitor_SMD:C_0201_0603Metric"
+		(property "Footprint" "Resistor_SMD:R_0201_0603Metric"
 			(at 59.69 44.958 90)
 			(hide yes)
@@
 		)
 		(instances
-			(project "resolution_w7"
+			(project "ATTiny1616-S"
 				(path "/ee73a050-21e3-4389-9e79-fb5dbee0e802"
 					(reference "R1")
@@
 		)
 		(instances
-			(project "resolution_w7"
+			(project "ATTiny1616-S"
 				(path "/ee73a050-21e3-4389-9e79-fb5dbee0e802"
 					(reference "#PWR07")
@@
 			)
 		)
-		(property "Footprint" "Capacitor_SMD:C_0201_0603Metric"
+		(property "Footprint" "Resistor_SMD:R_0201_0603Metric"
 			(at 66.04 104.648 90)
 			(hide yes)
@@
 		)
 		(instances
-			(project "resolution_w7"
+			(project "ATTiny1616-S"
 				(path "/ee73a050-21e3-4389-9e79-fb5dbee0e802"
 					(reference "R3")
@@
 		)
 		(instances
-			(project "resolution_w7"
+			(project "ATTiny1616-S"
 				(path "/ee73a050-21e3-4389-9e79-fb5dbee0e802"
 					(reference "#PWR027")
@@
 		)
 		(instances
-			(project "resolution_w7"
+			(project "ATTiny1616-S"
 				(path "/ee73a050-21e3-4389-9e79-fb5dbee0e802"
 					(reference "C2")
@@
 		)
 		(instances
-			(project "resolution_w7"
+			(project "ATTiny1616-S"
 				(path "/ee73a050-21e3-4389-9e79-fb5dbee0e802"
 					(reference "#PWR012")
@@
 		)
 		(instances
-			(project "resolution_w7"
+			(project "ATTiny1616-S"
 				(path "/ee73a050-21e3-4389-9e79-fb5dbee0e802"
 					(reference "U3")
@@
 		)
 		(instances
-			(project "resolution_w7"
+			(project "ATTiny1616-S"
 				(path "/ee73a050-21e3-4389-9e79-fb5dbee0e802"
 					(reference "#PWR08")
@@
 		)
 		(instances
-			(project "resolution_w7"
+			(project "ATTiny1616-S"
 				(path "/ee73a050-21e3-4389-9e79-fb5dbee0e802"
 					(reference "#PWR024")
@@
 		)
 		(instances
-			(project "resolution_w7"
+			(project "ATTiny1616-S"
 				(path "/ee73a050-21e3-4389-9e79-fb5dbee0e802"
 					(reference "#PWR010")
@@
 		)
 		(instances
-			(project "resolution_w7"
+			(project "ATTiny1616-S"
 				(path "/ee73a050-21e3-4389-9e79-fb5dbee0e802"
 					(reference "#PWR011")
@@
 		)
 		(instances
-			(project "resolution_w7"
+			(project "ATTiny1616-S"
 				(path "/ee73a050-21e3-4389-9e79-fb5dbee0e802"
 					(reference "#PWR013")
@@
 		)
 		(instances
-			(project "resolution_w7"
+			(project "ATTiny1616-S"
 				(path "/ee73a050-21e3-4389-9e79-fb5dbee0e802"
 					(reference "#PWR026")
@@
 		)
 		(instances
-			(project "resolution_w7"
+			(project "ATTiny1616-S"
 				(path "/ee73a050-21e3-4389-9e79-fb5dbee0e802"
 					(reference "#PWR02")
@@
 		)
 		(instances
-			(project "resolution_w7"
+			(project "ATTiny1616-S"
 				(path "/ee73a050-21e3-4389-9e79-fb5dbee0e802"
 					(reference "#PWR014")
@@
 		)
 		(instances
-			(project "resolution_w7"
+			(project "ATTiny1616-S"
 				(path "/ee73a050-21e3-4389-9e79-fb5dbee0e802"
 					(reference "#PWR022")
@@
 		)
 		(instances
-			(project "resolution_w7"
+			(project "ATTiny1616-S"
 				(path "/ee73a050-21e3-4389-9e79-fb5dbee0e802"
 					(reference "#PWR05")
@@
 		)
 		(instances
-			(project "resolution_w7"
+			(project "ATTiny1616-S"
 				(path "/ee73a050-21e3-4389-9e79-fb5dbee0e802"
 					(reference "#PWR04")
@@
 		)
 		(instances
-			(project "resolution_w7"
+			(project "ATTiny1616-S"
 				(path "/ee73a050-21e3-4389-9e79-fb5dbee0e802"
 					(reference "#PWR021")
@@
 		)
 		(instances
-			(project "resolution_w7"
+			(project "ATTiny1616-S"
 				(path "/ee73a050-21e3-4389-9e79-fb5dbee0e802"
 					(reference "U2")
@@
 		)
 		(instances
-			(project "resolution_w7"
+			(project "ATTiny1616-S"
 				(path "/ee73a050-21e3-4389-9e79-fb5dbee0e802"
 					(reference "#PWR03")
@@
 		)
 		(instances
-			(project "resolution_w7"
+			(project "ATTiny1616-S"
 				(path "/ee73a050-21e3-4389-9e79-fb5dbee0e802"
 					(reference "#PWR016")
@@
 		)
 		(instances
-			(project "resolution_w7"
+			(project "ATTiny1616-S"
 				(path "/ee73a050-21e3-4389-9e79-fb5dbee0e802"
 					(reference "D1")
@@
 		)
 		(instances
-			(project "resolution_w7"
+			(project "ATTiny1616-S"
 				(path "/ee73a050-21e3-4389-9e79-fb5dbee0e802"
 					(reference "C4")
@@
 		)
 		(instances
-			(project "resolution_w7"
+			(project "ATTiny1616-S"
 				(path "/ee73a050-21e3-4389-9e79-fb5dbee0e802"
 					(reference "#PWR06")
